File: Board/Switch Panel Rev 1/Switch Panel Rev 1.kicad_sch (KiCad schematic)
At the start: 0 parts

Commit message: Board Updates
Other:
- added sheet Connector (Connector.kicad_sch)
Changed lines of the file:
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@@
+    )
+  )
+  (sheet (at 43.18 64.77) (size 31.75 20.32) (fields_autoplaced)
+    (stroke (width 0.1524) (type solid))
+    (fill (color 0 0 0 0.0000))
+    (property "Sheetname" "Connector" (at 43.18 64.0584 0)
+      (effects (font (size 1.27 1.27)) (justify left bottom))
+    )
+    (property "Sheetfile" "Connector.kicad_sch" (at 43.18 85.6746 0)
+      (effects (font (size 1.27 1.27)) (justify left top))
+    )
+    (instances
+      (project "Switch Panel Rev 1"
+        (path "/6f128f22-9cbc-4f0e-a584-e54a559c0e90" (page "6"))
+      )
     )
   )
