File: Board/Switch Panel Rev 1/Switch Panel Rev 1.kicad_pcb (KiCad board)
At the start: 2 copper layers, 120.7 x 57.1 mm, 51 parts, among them J1 Conn_ARM_SWD_TagConnect_TC203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, J2 USB_C_Receptacle_USB2.0, U1 STM32G491CEUx, U2 MB85RS64, U3 LMR50410Y5FQDBVRQ1, U4 TPS2116DRLR, U5 AP2112K-3.3, U6 MCP2558FD-xMF, Y1 8MHz, Y2 32.768kHz

Commit message: Board work
Parts:
- added C20: 0.1uF, Capacitor_SMD:C_0603_1608Metric_Pad1.08x0.95mm_HandSolder, F.Cu at (144.2, 48.1)
- added C21: 0.1uF, Capacitor_SMD:C_0603_1608Metric_Pad1.08x0.95mm_HandSolder, F.Cu at (112.4, 48.1)
- added C22: 0.1uF, Capacitor_SMD:C_0603_1608Metric_Pad1.08x0.95mm_HandSolder, F.Cu at (80.7, 48.1)
- added C23: 0.1uF, Capacitor_SMD:C_0603_1608Metric_Pad1.08x0.95mm_HandSolder, F.Cu at (48.9, 48.1)
- added C24: 0.1uF, Capacitor_SMD:C_0603_1608Metric_Pad1.08x0.95mm_HandSolder, F.Cu at (144.2, 79.8)
- added C25: 0.1uF, Capacitor_SMD:C_0603_1608Metric_Pad1.08x0.95mm_HandSolder, F.Cu at (112.4, 79.8)
- added C26: 0.1uF, Capacitor_SMD:C_0603_1608Metric_Pad1.08x0.95mm_HandSolder, F.Cu at (80.7, 79.8)
- added C27: 0.1uF, Capacitor_SMD:C_0603_1608Metric_Pad1.08x0.95mm_HandSolder, F.Cu at (48.9, 79.8)
- added REF**: MountingHole_3.2mm_M3_DIN965, MountingHole:MountingHole_3.2mm_M3_DIN965, F.Cu at (66.7, 41.3)
- added REF**1: MountingHole_3.2mm_M3_DIN965, MountingHole:MountingHole_3.2mm_M3_DIN965, F.Cu at (98.4, 41.3)
- added REF**2: MountingHole_3.2mm_M3_DIN965, MountingHole:MountingHole_3.2mm_M3_DIN965, F.Cu at (130.2, 41.3)
- added REF**3: MountingHole_3.2mm_M3_DIN965, MountingHole:MountingHole_3.2mm_M3_DIN965, F.Cu at (66.7, 92.1)
- added REF**4: MountingHole_3.2mm_M3_DIN965, MountingHole:MountingHole_3.2mm_M3_DIN965, F.Cu at (98.4, 92.1)
- added REF**5: MountingHole_3.2mm_M3_DIN965, MountingHole:MountingHole_3.2mm_M3_DIN965, F.Cu at (130.2, 92.1)
- added U16: SN74LV1T34DBV, Package_TO_SOT_SMD:SOT-23-5, F.Cu at (65.8, 134.4)
- U10, U11, U12, U13, U14, U7, U8, U9: footprint MyKiCadLibraries:SW_Cherry_MX_Plate_RGB -> MyKiCadLibraries:SW_Kailh_Choc_RGB
- moved U2 75.1 mm to (64.2, 56.9), turned to 180 degrees
- moved C6 74.9 mm to (54.0, 59.5)
- moved C11 73.3 mm to (63.9, 60.5)
- moved FB1 72.4 mm to (54.0, 61.0), turned to 180 degrees
- moved Y1 71.5 mm to (61.6, 64.9), turned to 90 degrees
- moved Y2 70.7 mm to (61.7, 69.8), turned to 90 degrees
- moved C9 68.0 mm to (54.0, 58.0)
- moved C2 65.7 mm to (65.6, 64.1), turned to 180 degrees
- moved C4 65.7 mm to (65.0, 68.9), turned to 180 degrees
- moved R4 63.7 mm to (47.9, 65.7)
- moved U5 63.6 mm to (72.5, 66.7), turned to 90 degrees
- moved C1 62.3 mm to (65.6, 65.5), turned to 180 degrees
- moved R7 62.2 mm to (75.0, 70.5), turned to -90 degrees
- moved C3 62.2 mm to (65.0, 70.3), turned to 180 degrees
- moved C5 60.9 mm to (48.7, 70.1), turned to 90 degrees
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Connections:
- U1 pad 28: Sw7 -> RGB_DI
- U1 pad 8: unconnected-(U1-PA0-Pad8) -> Sw7
- U7 pad 4: unconnected-(U7-DI-Pad4) -> Net-(U16-Y)
Routing:
- net GND: track 0.00 -> 61.4 mm, vias 0 -> 56
- net +3.3V: track 0.00 -> 52.5 mm, vias 0 -> 12
- net Usb 5V: track 0.00 -> 48.4 mm, vias 0 -> 4
- net +5V: track 0.00 -> 29.9 mm, vias 0 -> 12
- net /Mcu/SPI1_SS_Memory: track 0.00 -> 21.4 mm
- net /Mcu/Memory_Wp: track 0.00 -> 18.5 mm
- net CanSilent: track 0.00 -> 16.3 mm
- net SPI1_Miso: track 0.00 -> 16.1 mm
- net /Mcu/SWO: track 0.00 -> 14.7 mm
- net Regulated 5V: track 0.00 -> 14.2 mm
- net /Mcu/SWCLK: track 0.00 -> 12.5 mm
- net /Mcu/SWDIO: track 0.00 -> 12.1 mm
- net CanTx: track 0.00 -> 11.9 mm
- net SPI1_Mosi: track 0.00 -> 10.9 mm
- net /Mcu/Usb D-: track 0.00 -> 9.96 mm
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- added copper zone on F.Cu, net +3.3V
- added copper zone on In2.Cu, net +3.3V
- added copper zone on F.Cu, net +5V
- added copper zone on In2.Cu, net +5V
- added copper zone on F.Cu, net /Mcu/Usb_Shield
- added copper zone on In1.Cu, net GND
- added copper zone on F.Cu, net Ignition
- added copper zone on F.Cu, net Net-(U3-SW)
- added copper zone on F.Cu, net Regulated 5V
Other:
- outline, holes or cut-outs redrawn
- copper layers 2 -> 4

Commit message: Board Updates
Parts:
- added J3: Conn_01x04, MyKiCadLibraries:Tie Wrap Connector, F.Cu at (82.0, 66.7)
- moved U14 100.4 mm to (146.1, 50.8)
- moved C27 100.4 mm to (144.2, 48.1)
- moved U7 95.3 mm to (50.8, 50.8)
- moved C20 95.2 mm to (48.9, 48.1)
- moved D1 92.1 mm to (60.1, 49.0)
- moved R1 88.9 mm to (60.1, 50.4)
- moved U16 81.3 mm to (47.2, 55.3), turned to 90 degrees
- moved S2 76.0 mm to (69.1, 49.7), turned to 90 degrees
- moved R2 73.6 mm to (69.2, 53.3)
- moved C21 71.0 mm to (48.9, 79.8)
- moved U9 71.0 mm to (50.8, 82.5)
- moved S1 70.9 mm to (64.5, 49.7), turned to 90 degrees
- moved C26 63.5 mm to (144.2, 79.8)
- moved U12 63.5 mm to (146.1, 82.5)
- moved U8 44.9 mm to (114.3, 50.8)
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Connections:
- R1 pad 1: unconnected-(R1-Pad1) -> /Mcu/User_Led
- U1 pad 10: unconnected-(U1-PA2-Pad10) -> Sw4
- U1 pad 11: unconnected-(U1-PA3-Pad11) -> PowerSwitchStatus
- U1 pad 18: unconnected-(U1-PB1-Pad18) -> /Mcu/User_Led
- U1 pad 19: PowerSwitchStatus -> unconnected-(U1-PB2-Pad19)
- U1 pad 22: Sw2 -> unconnected-(U1-PB10-Pad22)
- U1 pad 24: Sw3 -> unconnected-(U1-PB11-Pad24)
- U1 pad 25: Sw4 -> unconnected-(U1-PB12-Pad25)
- U1 pad 26: Sw5 -> unconnected-(U1-PB13-Pad26)
- U1 pad 27: Sw6 -> Sw1
- U1 pad 38: Sw8 -> Sw6
- U1 pad 39: unconnected-(U1-PC10-Pad39) -> Sw7
- U1 pad 40: unconnected-(U1-PC11-Pad40) -> Sw8
- U1 pad 42: unconnected-(U1-PB4-Pad42) -> Sw2
- U1 pad 47: Sw1 -> unconnected-(U1-PB9-Pad47)
- U1 pad 8: Sw7 -> Sw3
- U1 pad 9: unconnected-(U1-PA1-Pad9) -> Sw5
Routing:
- net Sw7: track 0.00 -> 119.0 mm, vias 0 -> 1
- net Sw8: track 0.00 -> 108.4 mm, vias 0 -> 1
- net Sw6: track 0.00 -> 88.7 mm, vias 0 -> 1
- net Net-(U11-DI): track 0.00 -> 66.2 mm
- net Sw5: track 0.00 -> 61.5 mm, vias 0 -> 1
- net Net-(U10-DO): track 0.00 -> 52.3 mm
- net /Mcu/RESET: track 0.00 -> 50.1 mm, vias 0 -> 3
- net Sw3: track 0.00 -> 49.7 mm
- net Net-(U7-DO): track 0.00 -> 48.6 mm, vias 0 -> 2
- net Can-: track 0.00 -> 45.9 mm, vias 0 -> 1
- net Net-(U13-DO): track 0.00 -> 44.5 mm
- net Can+: track 0.00 -> 43.0 mm, vias 0 -> 1
- net Net-(U10-DI): track 0.00 -> 41.3 mm
- net Net-(U11-DO): track 0.00 -> 35.5 mm
- net Net-(U12-DO): track 0.00 -> 32.4 mm
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- added copper zone on B.Cu, net GND
- added copper zone on F.Cu, net GND
Other:
- board text added: "+12V"
- board text added: "Boot_0"
- board text added: "CanHi"
- board text added: "CanLo"
- board text added: "Gnd"
- board text added: "Reset"

Commit message: Added output files and bom file
Parts:
- removed REF**5: MountingHole_3.2mm_M3_DIN965, MountingHole:MountingHole_3.2mm_M3_DIN965
- added G***: LOGO, Bryan_Lib:Brytec_Logo, F.Cu at (139.1, 66.7)
- added REF**4: MountingHole_3.2mm_M3_DIN965, MountingHole:MountingHole_3.2mm_M3_DIN965, F.Cu at (130.2, 92.1)
Other:
- board text added: "Switch Panel - Rev 1 2023"
